File: Spi2Dcc/SpiDcc.kicad_pcb (KiCad board)
At the start: 2 copper layers, 100 x 65 mm, 90 parts, among them P701 LED, P702 Invld cmd out, P703 Mstr SW, P704 Mstr SW bypass, P705 Bstr En Out, P706 Mstr SW out, P801 SPI, P901 Bstr 1, P902 Bstr 2, P903 Bstr 3, P904 Bstr 4, Q701 BC327-40, Q702 BC327-40, Q703 BC327-40, Q901 BC327-40, U201 LM555N, U202 74HC74, U301 74HC4053, U302 74HC32, U401 74HC163, U402 74HC04, U403 74HC163, U404 74HC193, U501 74HC590, U502 74HC75, U503 74HC153, U601 74HC595, U602 74HC165, U603 74HC595, U604 74HC165, U605 74HC595, U606 74HC165, U607 74HC595, U608 74HC165, U609 74HC595, U610 74HC165, U611 74HC595, U612 74HC165

Commit message: Set solder mask clearance and minimum width as specified by Elecrow to 0.2
Other:
- rule pad_to_mask_clearance: 0 -> 0.2
- rule solder_mask_min_width: 0.3 -> 0.2
Changed lines of the file:
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@@
     (links 349)
     (no_connects 0)
-    (area 99.865 84.210285 200.050001 150.050001)
+    (area 99.949999 84.949999 200.050001 150.050001)
     (thickness 1.6)
     (drawings 68)
@@
     (pad_size 5 5)
     (pad_drill 3.2)
-    (pad_to_mask_clearance 0)
-    (solder_mask_min_width 0.3)
+    (pad_to_mask_clearance 0.2)
+    (solder_mask_min_width 0.2)
     (aux_axis_origin 0 0)
     (visible_elements 7FFFFFFF)
