File: Spi2Dcc/ShiftRegisters.sch (KiCad schematic (older format))
At the start: 24 parts, among them U601 74HC595, U602 74HC165, U603 74HC595, U604 74HC165, U605 74HC595, U606 74HC165, U607 74HC595, U608 74HC165, U609 74HC595, U610 74HC165, U611 74HC595, U612 74HC165

Commit message: fix command length bits swapped. Connect mounting hole pads to GND.
Parts:
- U601, U603, U605, U607, U609, U611: footprint (none) -> SMD_Packages:SO-16-N
Changed lines of the file:
@@
 F 0 "U601" H 2000 5550 50  0000 C CNN
 F 1 "74HC595" H 1850 4350 50  0000 C CNN
-F 2 "" H 1850 4950 50  0000 C CNN
+F 2 "SMD_Packages:SO-16-N" H 1850 4950 50  0001 C CNN
 F 3 "" H 1850 4950 50  0000 C CNN
 	1    1850 4950
@@
 F 0 "U603" H 3700 5550 50  0000 C CNN
 F 1 "74HC595" H 3550 4350 50  0000 C CNN
-F 2 "" H 3550 4950 50  0000 C CNN
+F 2 "SMD_Packages:SO-16-N" H 3550 4950 50  0001 C CNN
 F 3 "" H 3550 4950 50  0000 C CNN
 	1    3550 4950
@@
 F 0 "U605" H 5400 5550 50  0000 C CNN
 F 1 "74HC595" H 5250 4350 50  0000 C CNN
-F 2 "" H 5250 4950 50  0000 C CNN
+F 2 "SMD_Packages:SO-16-N" H 5250 4950 50  0001 C CNN
 F 3 "" H 5250 4950 50  0000 C CNN
 	1    5250 4950
@@
 F 0 "U607" H 7100 5550 50  0000 C CNN
 F 1 "74HC595" H 6950 4350 50  0000 C CNN
-F 2 "" H 6950 4950 50  0000 C CNN
+F 2 "SMD_Packages:SO-16-N" H 6950 4950 50  0001 C CNN
 F 3 "" H 6950 4950 50  0000 C CNN
 	1    6950 4950
@@
 F 0 "U609" H 8800 5550 50  0000 C CNN
 F 1 "74HC595" H 8650 4350 50  0000 C CNN
-F 2 "" H 8650 4950 50  0000 C CNN
+F 2 "SMD_Packages:SO-16-N" H 8650 4950 50  0001 C CNN
 F 3 "" H 8650 4950 50  0000 C CNN
 	1    8650 4950
@@
 F 0 "U611" H 10550 5550 50  0000 C CNN
 F 1 "74HC595" H 10400 4350 50  0000 C CNN
-F 2 "" H 10400 4950 50  0000 C CNN
+F 2 "SMD_Packages:SO-16-N" H 10400 4950 50  0001 C CNN
 F 3 "" H 10400 4950 50  0000 C CNN
 	1    10400 4950
