File: FlexSensor/SPI.sch (KiCad schematic (older format))
At the start: 8 parts

Commit message: Introduced the analog input selector.
Parts:
- added U?: 74HC04, symbol 74xx:74HC04
Connections:
- net labels added: ADR6
- wire segments 39 -> 40
- no-connect marks 2 -> 3
Changed lines of the file:
@@
 $Descr A4 11693 8268
 encoding utf-8
-Sheet 3 3
+Sheet 3 5
 Title ""
 Date ""
@@
 $Comp
 L 74xx:74LS393 U?
-U 1 1 5AE447ED
+U 2 1 5AE447ED
 P 3000 2300
 F 0 "U?" H 3000 2667 50  0000 C CNN
@@
 F 2 "" H 3000 2300 50  0001 C CNN
 F 3 "74xx\\74LS393.pdf" H 3000 2300 50  0001 C CNN
-	1    3000 2300
+	2    3000 2300
 	1    0    0    -1
 $EndComp
@@
 $Comp
 L 74xx:74LS393 U?
-U 2 1 5AE448EE
+U 1 1 5AE448EE
 P 4250 2900
 F 0 "U?" H 4250 3267 50  0000 C CNN
@@
 F 2 "" H 4250 2900 50  0001 C CNN
 F 3 "74xx\\74LS393.pdf" H 4250 2900 50  0001 C CNN
-	2    4250 2900
-	1    0    0    -1
-$EndComp
-$Comp
-L 74xx:74LS393 U?
-U 1 1 5AE44A24
+	1    4250 2900
+	1    0    0    -1
+$EndComp
+$Comp
+L 74xx:74LS393 U?
+U 2 1 5AE44A24
 P 5450 3550
 F 0 "U?" H 5450 3917 50  0000 C CNN
@@
 F 2 "" H 5450 3550 50  0001 C CNN
 F 3 "74xx\\74LS393.pdf" H 5450 3550 50  0001 C CNN
-	1    5450 3550
+	2    5450 3550
 	1    0    0    -1
 $EndComp
@@
 L 74xx:74LS393 U?
 U 2 1 5AE44A2A
-P 6850 4150
-F 0 "U?" H 6850 4517 50  0000 C CNN
-F 1 "74HC393" H 6850 4426 50  0000 C CNN
-F 2 "" H 6850 4150 50  0001 C CNN
-F 3 "74xx\\74LS393.pdf" H 6850 4150 50  0001 C CNN
-	2    6850 4150
+P 3000 1200
+F 0 "U?" H 3000 1567 50  0000 C CNN
+F 1 "74HC393" H 3000 1476 50  0000 C CNN
+F 2 "" H 3000 1200 50  0001 C CNN
+F 3 "74xx\\74LS393.pdf" H 3000 1200 50  0001 C CNN
+	2    3000 1200
 	1    0    0    -1
 $EndComp
@@
 	4850 3450 4950 3450
 Wire Wire Line
-	5950 3750 6150 3750
-Wire Wire Line
-	6150 3750 6150 4050
-Wire Wire Line
-	6150 4050 6350 4050
-Wire Wire Line
-	1650 2500 2400 2500
-Wire Wire Line
 	2400 2500 2400 3100
 Wire Wire Line
@@
 Wire Wire Line
 	4850 3750 4950 3750
-Wire Wire Line
-	2500 2200 1650 2200
 Text Label 7400 2800 0    50   ~ 0
 ADR0
@@
 NoConn ~ 3500 2200
 NoConn ~ 3500 2300
-Wire Wire Line
-	3500 2500 3850 2500
-Wire Wire Line
-	3850 2500 3850 2000
-Wire Wire Line
-	3850 2000 4400 2000
+$Comp
+L 74xx:74HC04 U?
+U 1 1 5AE16C73
+P 1950 1100
+F 0 "U?" H 1950 1417 50  0000 C CNN
+F 1 "74HC04" H 1950 1326 50  0000 C CNN
+F 2 "" H 1950 1100 50  0001 C CNN
+F 3 "http://www.nxp.com/documents/data_sheet/74HC_HCT04.pdf" H 1950 1100 50  0001 C CNN
+	1    1950 1100
+	1    0    0    -1
+$EndComp
+Wire Wire Line
+	850  2200 1200 2200
+Wire Wire Line
+	1200 2200 1200 1100
+Wire Wire Line
+	1200 1100 1650 1100
+Connection ~ 1200 2200
+Wire Wire Line
+	1200 2200 2500 2200
+Wire Wire Line
+	850  2500 2400 2500
+Wire Wire Line
+	2400 2500 2400 1400
+Wire Wire Line
+	2400 1400 2500 1400
+Wire Wire Line
+	2250 1100 2500 1100
+Wire Wire Line
+	5950 3750 7700 3750
+Entry Wire Line
+	7700 3750 7800 3850
+Text Label 7400 3750 0    50   ~ 0
+ADR6
+NoConn ~ 3500 2500
 Wire Bus Line
 	7800 2750 7800 4350
