File: FlexSensor/FlexSensor.sch (KiCad schematic (older format))
At the start: 0 parts

Commit message: Introduced the analog input selector.
Parts:
- added C? (x2): 100nF, symbol Device:C
- added C? (x9): 100nF, symbol Device:C_Small
- added D? (x2): 1N5821, Diode_THT:D_DO-201AD_P15.24mm_Horizontal, symbol Diode:1N5821
- added D? (x4): 1N4148, Diode_THT:D_DO-35_SOD27_P7.62mm_Horizontal, symbol Diode:1N4148
- added D?: LED_CRGB, symbol Device:LED_CRGB
- added J?: S88_IN, symbol Connector:Conn_01x06_Male
- added J?: S88-N_IN, symbol Connector:RJ45
- added J?: S88_OUT, symbol Connector:Conn_01x06_Male
- added J?: S88-N_OUT, symbol Connector:RJ45
- added J?: BankH, symbol Connector:Screw_Terminal_01x08
- added J?: BankG, symbol Connector:Screw_Terminal_01x08
- added J?: BankF, symbol Connector:Screw_Terminal_01x08
- added J?: BankE, symbol Connector:Screw_Terminal_01x08
- added J?: BankA, symbol Connector:Screw_Terminal_01x08
- added J?: BankB, symbol Connector:Screw_Terminal_01x08
- added J?: BankC, symbol Connector:Screw_Terminal_01x08
- added J?: BankD, symbol Connector:Screw_Terminal_01x08
- added R? (x10): 36K, symbol Device:R
- added R? (x11): R, symbol Device:R
- added R?: 4.7K, symbol Device:R
- added R? (x4): 10K, symbol Device:R
- added R?: R_PHOTO, symbol Device:R_PHOTO
- added R?: 620K, symbol Device:R
- added R?: 100K, symbol Device:R
- added R?: 150K, symbol Device:R
- added SW?: SW_Push, symbol Switch:SW_Push
- added U? (x8): LM339, symbol Comparator:LM339
- added U? (x9): CD4051B, symbol 4xxx:4051
- added U?: ULN2003A, symbol Transistor_Array:ULN2003A
- added U? (x2): LM6132, symbol Amplifier_Operational:LM358
Connections:
- new net: C?.1, C?.1, D?.1 (K), D?.1 (K), R?.1, R?.1, U?.3 (V+), U?.3 (V+)
- new net: D?.1 (K), U?.4 (-) (x3)
- new net: R?.1, R?.2, U?.4 (-), U?.5 (+), U?.5 (+)
- new net: J?.1 (Pin_1), J?.2, R?.2, U?.2
- new net: D?.2 (A), J?.3 (Pin_3), J?.4
- new net: D?.2 (A), J?.4 (Pin_4), J?.6
- new net: J?.5 (Pin_5), J?.7
- new net: D?.2 (A), J?.1, J?.6 (Pin_6)
- new net: D?.2 (A), J?.8
- new net: R?.1, R?.2, U?.5 (+), U?.5 (+), U?.5 (+), U?.5 (+), U?.5 (+)
- new net: J?.4 (Pin_4), J?.6, R?.2, U?.2
- new net: J?.3 (Pin_3), J?.4, R?.2, U?.2
- new net: J?.8, R?.2, U?.2
- new net: D?.1 (K), U?.5 (+)
- new net: J?.5 (Pin_5), J?.7, R?.2, U?.2
- new net: D?.2 (A), J?.1 (Pin_1), J?.2
- new net: D?.2 (RA), R?.1
- new net: D?.3 (GA), R?.1
- new net: D?.4 (BA), R?.1
- new net: J?.5 (Pin_5), U?.1 (X4) (x8)
- new net: J?.4 (Pin_4), U?.12 (X3) (x8)
- new net: J?.1 (Pin_1), U?.13 (X0) (x8)
- new net: J?.2 (Pin_2), U?.14 (X1) (x8)
- new net: J?.3 (Pin_3), U?.15 (X2) (x8)
- new net: J?.7 (Pin_7), U?.2 (X6) (x8)
- new net: U?.3 (X), U?.4 (X7)
- new net: J?.8 (Pin_8), U?.4 (X7) (x8)
- new net: J?.6 (Pin_6), U?.5 (X5) (x8)
- new net: U?.2 (X6), U?.3 (X)
- new net: U?.3 (X), U?.5 (X5)
- new net: U?.1 (X4), U?.3 (X)
- new net: U?.12 (X3), U?.3 (X)
- new net: U?.15 (X2), U?.3 (X)
- new net: U?.14 (X1), U?.3 (X)
- new net: U?.13 (X0), U?.3 (X)
- new net: R?.2, U?.10 (O7)
- new net: R?.2, U?.11 (O6)
- new net: R?.2, U?.12 (O5)
- new net: R?.2, U?.13 (O4)
- new net: R?.2, U?.14 (O3)
- new net: R?.2, U?.15 (O2)
- new net: R?.2, U?.16 (O1)
- new net: R?.1, R?.2, U?.3 (+)
- new net: R?.1, U?.1
- new net: R?.2, U?.2 (-)
- new net: R?.1, R?.2
- new net +3V3: R?.1, R?.1, R?.1, R?.1, R?.1, R?.2, R?.2
- new net +5V: D?.2 (A), J?.1, J?.6 (Pin_6), R?.1, R?.1, R?.1, R?.1
- new net ADR0: U?.1 (I1)
- new net ADR0_VDD: U?.11 (A), U?.11 (A), U?.11 (A), U?.11 (A), U?.11 (A), U?.11 (A), U?.11 (A), U?.11 (A)
- new net ADR1: U?.2 (I2)
- new net ADR1_VDD: U?.10 (B), U?.10 (B), U?.10 (B), U?.10 (B), U?.10 (B), U?.10 (B), U?.10 (B), U?.10 (B)
- new net ADR2: U?.3 (I3)
- new net ADR2_VDD: U?.9 (C), U?.9 (C), U?.9 (C), U?.9 (C), U?.9 (C), U?.9 (C), U?.9 (C), U?.9 (C)
- new net ADR3: U?.4 (I4)
- new net ADR3_VDD: U?.11 (A)
- new net ADR4: U?.5 (I5)
- new net ADR4_VDD: U?.10 (B)
- new net ADR5: U?.6 (I6)
- new net ADR5_VDD: U?.9 (C)
- new net ANALOG: R?.1, R?.1, U?.3 (X)
- new net GND: C?.2, C?.2, C?.2, C?.2, C?.2, C?.2, C?.2, C?.2, C?.2, C?.2, C?.2, D?.1 (K), J?.2 (Pin_2), J?.2 (Pin_2), J?.3, J?.3, J?.5, J?.5, R?.2, R?.2, R?.2, R?.2, R?.2, SW?.2, U?.12 (V-), U?.12 (V-), U?.6 (Inh), U?.6 (Inh), U?.6 (Inh), U?.6 (Inh), U?.6 (Inh), U?.6 (Inh), U?.6 (Inh), U?.6 (Inh), U?.6 (Inh), U?.7 (VEE), U?.7 (VEE), U?.7 (VEE), U?.7 (VEE), U?.7 (VEE), U?.7 (VEE), U?.7 (VEE), U?.7 (VEE), U?.7 (VEE), U?.8 (GND), U?.8 (VSS), U?.8 (VSS), U?.8 (VSS), U?.8 (VSS), U?.8 (VSS), U?.8 (VSS), U?.8 (VSS), U?.8 (VSS), U?.8 (VSS)
- new net LED_B: R?.2
- new net LED_G: R?.2
- new net LED_R: R?.2
- new net PHOTO_SENSOR: R?.1, R?.1
- new net PULL_DOWN: U?.7 (I7)
- new net VDD: C?.1, C?.1, C?.1, C?.1, C?.1, C?.1, C?.1, C?.1, C?.1, R?.1, R?.1, R?.1, R?.1, R?.1, R?.1, U?.16 (VDD), U?.16 (VDD), U?.16 (VDD), U?.16 (VDD), U?.16 (VDD), U?.16 (VDD), U?.16 (VDD), U?.16 (VDD), U?.16 (VDD)
- new net ~BUTTON: R?.1, SW?.1
- new net ~S88_IN_CLK: R?.2, U?.2
- new net ~S88_IN_DATA: U?.4 (-)
- new net ~S88_IN_LOAD: R?.2, U?.2
- new net ~S88_OUT_CLK: U?.4 (-)
- new net ~S88_OUT_DATA: R?.2, U?.2
- new net ~S88_OUT_LOAD: U?.4 (-)
- new net ~S88_OUT_RESET: U?.4 (-)
- no-connect marks 0 -> 1
Other:
- note added: "Add capacitor to drive interrupt pin?"
- note added: "Buffer to get rid of pull up that might\nfight upstream pull down?"
- note added: "Cheap level shifter without pullup?"
- note added: "Demultiplexer"
- note added: "Power the opamp at S88 V+ - diode drop,\nmaintaining 5V - diode drop if S88 is not\npowered."
- note added: "Replace with internal pull up/down?\nTake debounce capacitor value from ESP32 reference dev kit scematic?\nIf using dev board, not needed - already contains two buttons\nIf not using dev board - do I also need two buttons?"
- note added: "S88"
- note added: "TODO:\n- LocoNet support: http://locobuffer.com/ (PL2303 is a lot cheaper, investigate)\n- Level shifting in S88 with transistors?\n- Two way communication on RAILDATA in S88\n- Analog inputs\n- ESP32 (dev board for now, or consider the MAX322/PL2303 and make it all on board now)\n- Break out remaining pins for extra GPIO/UART/SPI/I2C\n-- Level shift to 5V - room on the board?\n"
- note added: "ULN2803A could drive a second pull down,\nfor 3 different pull down values \nusing one extra GPIO pin."
- note added: "Use two times dac to allow add/subtract before hitting ADC. \nConsider support additional scaling? \nFeed opamps 3.3V to avoid overshooting the analog input"

Commit message: Added initial analog input.
Parts:
- removed R?: R, symbol Device:R
- removed R?: 150K, symbol Device:R
- removed R?: 10K, symbol Device:R
- added C?: 100µF, symbol Device:CP
- added C?: 4.7µF, symbol Device:CP
- added C? (x5): 100nF, symbol Device:C_Small
- added C? (x4): 10uF, symbol Device:CP
- added C?: NC (2.2uF), symbol Device:CP
- added C? (x6): NC, symbol Device:C_Small
- added J?: 12-20VDC, symbol Connector:Screw_Terminal_01x02
- added J?: USB_B_Micro, symbol Connector:USB_B_Micro
- added Q?: FQP47P06, Package_TO_SOT_THT:TO-220-3_Vertical, symbol Transistor_FET:IRF9540N
- added R? (x6): 10K, symbol Device:R
- added R? (x2): 180K, symbol Device:R
- added R?: 36K, symbol Device:R
- added TP? (x7): Test_Point, symbol Connector:Test_Point
- added U?: ICL7660, symbol Regulator_SwitchedCapacitor:ICL7660
- added U?: LD1117S33TR_SOT223, Package_TO_SOT_SMD:SOT-223-3_TabPin2, symbol Regulator_Linear:LD1117S33TR_SOT223
- added U? (x2): LM6132, symbol Amplifier_Operational:LM358
- added U?: LD1117S50TR_SOT223, Package_TO_SOT_SMD:SOT-223-3_TabPin2, symbol Regulator_Linear:LD1117S50TR_SOT223
- added U?: CP2102N-A01-GQFN24, Package_DFN_QFN:QFN-24-1EP_4x4mm_P0.5mm_EP2.6x2.6mm, symbol Interface_USB:CP2102N-A01-GQFN24
- R?: value 620K -> 820K
- R?: value 100K -> 68K
Connections:
- net +3V3: now also U?.8 (V+), C?.1, C?.1, C?.1, R?.2, U?.2 (VO), U?.8 (V+), U?.8 (V+)
- net +5V: now also C?.1, U?.2 (VO)
- net ANALOG: now also TP?.1
- net GND: now also C?.1, C?.2, C?.2, C?.2, C?.2, C?.2, C?.2, C?.2, C?.2, C?.2, C?.2, C?.2, C?.2, J?.2 (Pin_2), J?.5 (GND), J?.6 (Shield), Q?.1 (G), R?.2, R?.2, U?.3 (GND), U?.4 (V-)
- net VDD: now also C?.1, C?.1, C?.1, C?.1, Q?.3 (S), U?.3 (VI), U?.3 (VI)
- net at R?.1, R?.2: now also U?.3 (+), C?.1, TP?.1; no longer U?.3 (+)
- net at U?.1: now also C?.1, R?.1, R?.2, TP?.1
- net at U?.2 (-): now also R?.1, R?.2
- net at U?.1: now also U?.2 (-), C?.1, R?.2, TP?.1
- net -3V3: now reaches U?.4 (V-)
- net -3V3: now also C?.1, C?.2, U?.5 (VOUT)
- new net: C?.1, U?.2 (CAP+)
- new net: C?.2, U?.4 (CAP-)
- new net: C?.1, U?.6 (LV)
- new net: C?.2, C?.2, U?.1 (GND) (x2)
- new net: J?.1 (Pin_1), Q?.2 (D)
- new net: R?.1, R?.1, U?.3 (+)
- new net: R?.1, R?.2, U?.2 (-) (x2)
- new net: R?.1, U?.3 (+)
- new net ANALOG_1x: C?.1, R?.1, TP?.1, U?.1, U?.3 (+)
- new net ANALOG_4.6x: C?.1, R?.1, TP?.1, U?.1
- new net ANALOG_OFFSET: C?.1, R?.2, TP?.1
- no-connect marks 1 -> 5
Other:
- note added: "+0.2V"
- note added: "-offset"
- note added: "0-1.6V"
- note added: "Attenuation"
- note added: "Power"
- note removed: "Use two times dac to allow add/subtract before hitting ADC. \nConsider support additional scaling? \nFeed opamps 3.3V to avoid overshooting the analog input"
- moved on the sheet: C?, D?, J?, R?, U?, U?A

Commit message: Redesigned S88, redesigned power, started to change all ESP32 pin allocations.
Parts:
- removed C?: 100nF, symbol Device:C
- removed C?: 100µF, symbol Device:CP
- removed C?: 4.7µF, symbol Device:CP
- removed C? (x2): 100nF, symbol Device:C_Small
- removed C? (x2): 10uF, symbol Device:CP
- removed C? (x3): NC, symbol Device:C_Small
- removed D? (x2): 1N5821, Diode_THT:D_DO-201AD_P15.24mm_Horizontal, symbol Diode:1N5821
- removed D? (x4): 1N4148, Diode_THT:D_DO-35_SOD27_P7.62mm_Horizontal, symbol Diode:1N4148
- removed J?: 12-20VDC, symbol Connector:Screw_Terminal_01x02
- removed J?: BankH, symbol Connector:Screw_Terminal_01x08
- removed J?: BankA, symbol Connector:Screw_Terminal_01x08
- removed J?: USB_B_Micro, symbol Connector:USB_B_Micro
- removed Q?: FQP47P06, Package_TO_SOT_THT:TO-220-3_Vertical, symbol Transistor_FET:IRF9540N
- removed R? (x5): 36K, symbol Device:R
- removed R? (x7): R, symbol Device:R
- removed R?: 4.7K, symbol Device:R
- removed R? (x2): 10K, symbol Device:R
- removed R?: R_PHOTO, symbol Device:R_PHOTO
- removed U? (x7): LM339, symbol Comparator:LM339
- removed U?: LD1117S33TR_SOT223, Package_TO_SOT_SMD:SOT-223-3_TabPin2, symbol Regulator_Linear:LD1117S33TR_SOT223
- removed U?: LD1117S50TR_SOT223, Package_TO_SOT_SMD:SOT-223-3_TabPin2, symbol Regulator_Linear:LD1117S50TR_SOT223
- removed U?: CP2102N-A01-GQFN24, Package_DFN_QFN:QFN-24-1EP_4x4mm_P0.5mm_EP2.6x2.6mm, symbol Interface_USB:CP2102N-A01-GQFN24
- added C? (x6): 100nF, symbol Device:C_Small
- added C?: 100μF, symbol Device:CP
- added C? (x4): 330nF, symbol Device:C_Small
- added C?: 1μF, symbol Device:CP
- added C?: 100µF, symbol Device:CP
- added C?: 4.7µF, symbol Device:CP
- added C? (x2): 22μF, symbol Device:C_Small
- added C?: 10μF, symbol Device:CP
- added C? (x2): 1nF, symbol Device:C_Small
- added C? (x3): NC, symbol Device:C_Small
- added C?: 100nF, symbol Device:C
- added D? (x4): 1N5821, Diode_THT:D_DO-201AD_P15.24mm_Horizontal, symbol Diode:1N5821
- added J?: 5-15VDC, symbol Connector:Screw_Terminal_01x02
- added J?: BankA, symbol Connector:Screw_Terminal_01x06
- added J?: BankH, symbol Connector:Screw_Terminal_01x06
- added L?: 22μH, symbol Device:L
- added Q? (x3): BC817, Package_TO_SOT_SMD:SOT-23, symbol Transistor_BJT:BC817
- added Q?: BC807, Package_TO_SOT_SMD:SOT-23, symbol Transistor_BJT:BC807
- added R? (x8): 10K, symbol Device:R
- added R? (x8): 270K, symbol Device:R
- added R? (x4): 27K, symbol Device:R
- added R? (x2): 470, symbol Device:R
- added R?: 470K, symbol Device:R
- added R?: 12K, symbol Device:R
- added R? (x2): ?, symbol Device:R
- added R?: 2.7K, symbol Device:R
- added SW?: RESET, symbol Switch:SW_Push
- added TP?: Test_Point, symbol Connector:Test_Point
- added U?: ESP32-WROOM, symbol Trainiot:ESP32-WROOM
- added U?: MT3608, symbol Trainiot:MT3608
- added U?: 74HC165, symbol Trainiot:74HC165
- added U?: LM78L05, symbol Trainiot:LM78L05
- added U?: LD1117S33TR_SOT223, Package_TO_SOT_SMD:SOT-223-3_TabPin2, symbol Regulator_Linear:LD1117S33TR_SOT223
- added U? (x3): 74HCT4053, symbol Trainiot:74HCT4053
- added U? (x3): LM339, symbol Comparator:LM339
- added U?: 74HC590, symbol 74xx:74HC590
- added U?: LM7820, Package_TO_SOT_THT:TO-220-3_Vertical, symbol Regulator_Linear:LM7805_TO220
- added U? (x7): 74HCT04, symbol 74xx:74HCT04
- added U?: 74HC595, symbol Trainiot:74HC595
- added U?: MCP42010, symbol Potentiometer_Digital:MCP42010
- C? (x2): value 10uF -> 10μF
- R?: value 10K -> 1K
Connections:
- net VDD is gone; now on net +3V3: C?.1, C?.1, C?.1, C?.1, C?.1, C?.1, C?.1, C?.1, C?.1, R?.1, R?.1, R?.1, R?.1, R?.1, R?.1, U?.16 (VDD), U?.16 (VDD), U?.16 (VDD), U?.16 (VDD), U?.16 (VDD), U?.16 (VDD), U?.16 (VDD), U?.16 (VDD), U?.16 (VDD)
- net ~BUTTON is gone; now on net GND: SW?.1
- net +3V3: now also U?.2 (X6), U?.3 (V+), U?.4 (X7), C?.1, C?.1, C?.1, C?.1, C?.1, C?.1, C?.1, C?.1, C?.1, C?.1, R?.1, R?.1, R?.1, R?.1, R?.2, R?.2, R?.2, R?.2, R?.2, U?.10 (SRCLR), U?.11 (~RS), U?.12 (1Y0), U?.12 (~SHDN), U?.14 (VDD), U?.16 (VCC), U?.16 (VCC), U?.16 (VCC), U?.16 (VDD), U?.16 (VDD), U?.16 (VDD), U?.2 (3V3), U?.2 (VO), U?.3 (VO), U?.8 (PA0)
- net +5V: now also C?.1, U?.14 (X1), C?.1, U?.1 (VO), U?.14 (VCC)
- net GND: now also U?.13 (X0), C?.2, C?.2, C?.2, C?.2, C?.2, C?.2, C?.2, C?.2, C?.2, C?.2, C?.2, C?.2, C?.2, C?.2, C?.2, C?.2, C?.2, C?.2, C?.2, C?.2, C?.2, J?.2 (Pin_2), Q?.3 (C), R?.1, R?.2, R?.2, R?.2, R?.2, R?.2, SW?.1, U?.1 (GND), U?.10 (PB0), U?.11, U?.12 (~CE), U?.13, U?.13 (1Y1), U?.13 (1Y1), U?.14 (~OE), U?.15 (GND), U?.2 (GND), U?.2 (GND), U?.38 (GND), U?.39 (GND-PAD), U?.4 (VSS), U?.7 (GND), U?.7 (VEE), U?.7 (VEE), U?.7 (VEE), U?.8 (GND), U?.8 (GND), U?.8 (GND), U?.8 (GND), U?.8 (GND), U?.8 (GND); no longer SW?.2
- net LED_B: now also U?.3 (QD)
- net LED_G: now also U?.2 (QC)
- net LED_R: now also U?.1 (QB)
- net PULL_DOWN: now also U?.4 (QE)
- net ~S88_IN_CLK: now also R?.1, R?.2, U?.10 (DS), U?.2
- net ~S88_IN_DATA: now also R?.2, R?.2, U?.6 (QG)
- net ~S88_IN_LOAD: now also R?.1, R?.2, U?.12 (D1), U?.2
- net ~S88_OUT_CLK: now also U?.3, U?.5 (QF)
- net ~S88_OUT_DATA: now also R?.1, R?.2, U?.11 (D0), U?.2
- net ~S88_OUT_LOAD: now also U?.5, U?.7 (QH)
- net ~S88_OUT_RESET: now also U?.9
- net at U?.4 (-): now also R?.1, R?.2
- net at J?.1 (Pin_1), J?.2: now also Q?.2 (E), Q?.2 (E)
- net at J?.3 (Pin_3), J?.4: now also R?.1, U?.5 (+)
- net at J?.4 (Pin_4), J?.6: now also R?.1, U?.5 (+)
- net at J?.1, J?.6 (Pin_6): now also Q?.3 (C)
- net at J?.8: now also U?.5 (+), R?.1
- net at J?.4 (Pin_4), J?.6: now also U?.6
- net at J?.3 (Pin_3), J?.4: now also U?.4
- net at J?.8: now also U?.2; no longer U?.2
- net at J?.5 (Pin_5), J?.7: now also U?.8
- net at J?.1 (Pin_1), J?.2: now also R?.1, U?.5 (+)
- net at U?.1 (X4): now also J?.5 (Pin_5)
- net at U?.12 (X3): now also J?.4 (Pin_4)
- net at U?.13 (X0): now also J?.1 (Pin_1)
- net at U?.14 (X1): now also J?.2 (Pin_2)
- net at U?.15 (X2): now also J?.3 (Pin_3)
- net at U?.5 (X5): now also J?.6 (Pin_6)
- net at U?.1 (X4): now also J?.3 (Pin_3)
- net at U?.12 (X3): now also J?.2 (Pin_2)
- net at U?.15 (X2): now also J?.1 (Pin_1)
- net at U?.2 (X6): now also J?.5 (Pin_5)
- net at U?.4 (X7): now also J?.6 (Pin_6)
- net at U?.5 (X5): now also J?.4 (Pin_4)
- net at R?.1, U?.3 (+): now also R?.2
- net at U?.4 (V-): now also R?.1
- net ADR0: no longer names the net of U?.1 (I1)
- net ADR0: now also U?.15 (Q0)
- net ADR1: no longer names the net of U?.2 (I2)
- net ADR1: now also U?.1 (Q1)
- net ADR2: no longer names the net of U?.3 (I3)
- net ADR2: now also U?.2 (Q2)
- net ADR3: no longer names the net of U?.4 (I4)
- net ADR3: now also U?.3 (Q3)
- net ADR4: no longer names the net of U?.5 (I5)
- net ADR4: now also U?.4 (Q4)
- net ADR5: no longer names the net of U?.6 (I6)
- net ADR5: now also U?.5 (Q5)
- net ANALOG_1x renamed ANALOG_1
- net ANALOG_4.6x renamed ANALOG_X
- net ANALOG_X: now also C?.1, U?.5 (PB1), U?.6 (PW1)
- net ANALOG_OFFSET: no longer names the net of R?.2, TP?.1
- net ANALOG_OFFSET: now also C?.1, U?.9 (PW0)
- new net: C?.1, R?.2, SW?.2 (x2)
- new net: D?.2 (A), J?.1 (Pin_1)
- new net: D?.2 (A), L?.2, U?.1 (SW)
- new net: R?.1, R?.2, U?.3 (FB)
- new net: C?.1, C?.1, C?.1, C?.1, D?.1 (K), D?.1 (K), L?.1, U?.3 (VI), U?.4 (EN), U?.5 (IN)
- new net: Q?.1 (B), R?.1 (x4)
- new net: Q?.3 (C), R?.1, U?.11 (S1), U?.13 (1Y1)
- new net: D?.1 (K), D?.2 (A)
- new net: C?.2, C?.2, U?.1 (GND)
- new net: R?.1, R?.2, U?.4 (-) (x3)
- new net: C?.1, R?.2, TP?.1, U?.7 (PA1)
- new net ANALOG_ATTENUATED: U?.4 (SENS_VP)
- new net BOOTING: U?.11 (S1), U?.12 (1Y0), U?.13 (G), U?.29 (IO5)
- new net BTN_AND_REVISION: R?.1, U?.14 (1Z), U?.5 (SENS_VN)
- new net DTR: Q?.2 (E), R?.2
- new net EN: Q?.3 (C), R?.1, U?.3 (EN)
- new net IO0: U?.14 (1Z), U?.25 (IO0)
- new net LOCONET_RX: U?.28 (IO17)
- new net LOCONET_TX: U?.27 (IO16)
- new net RMII_CRS_DV: U?.12 (IO27)
- new net RMII_EXT_OSC_CLK: U?.12 (1Y0)
- new net RMII_MDC: U?.37 (IO23)
- new net RMII_MDIO: U?.30 (IO18)
- new net RMII_RDX_0: U?.10 (IO25)
- new net RMII_RDX_1: U?.11 (IO26)
- new net RMII_TXD_0: U?.31 (IO19)
- new net RMII_TXD_1: U?.36 (IO22)
- new net RMII_TX_EN: U?.33 (IO21)
- new net RTS: Q?.2 (E), R?.2
- new net RXD0: U?.34 (RXD0)
- new net SPI_CLK: U?.11 (SRCLK), U?.2 (SCK), U?.23 (IO15)
- new net SPI_MOSI: U?.14 (SER), U?.16 (IO13)
- new net SPI_MOSI_2: U?.3 (SI), U?.9 (QH')
- new net SPI_SS: U?.11 (CPC), U?.13 (CPR), U?.14 (1Z)
- new net TXD0: U?.35 (TXD0)
- new net UART_CTS: U?.13 (IO14)
- new net UART_RTS: U?.14 (IO12)
- new net USB5V: D?.2 (A)
- new net ~ADR_RST: U?.10 (~MRC), U?.15 (QA)
- new net ~S88_TRACK: R?.1, R?.2, U?.1, U?.2
- new net ~SPI_SS: U?.1 (~CS), U?.11 (S1), U?.12 (RCLK), U?.24 (IO2)
- new net ~~24V: C?.1, C?.1, C?.1, D?.1 (K), R?.1, U?.1 (VI), U?.3 (VI)
- no-connect marks 5 -> 15
Other:
- note added: "Check diode choice\nin MT3608 datasheet"
- note added: "Figure out mosfet construction?\nIdeal external should "win" if 3V+"
- note added: "If gates are available,\ncould add reset and\n"present" if +5V detected"
- note added: "Inrush limit needed?"
- note added: "Single output, better scaling.\nConsider merging offset and scaling"
- note removed: "Add capacitor to drive interrupt pin?"
- note removed: "Buffer to get rid of pull up that might\nfight upstream pull down?"
- note removed: "Power the opamp at S88 V+ - diode drop,\nmaintaining 5V - diode drop if S88 is not\npowered."
- note removed: "Replace with internal pull up/down?\nTake debounce capacitor value from ESP32 reference dev kit scematic?\nIf using dev board, not needed - already contains two buttons\nIf not using dev board - do I also need two buttons?"
- note removed: "TODO:\n- LocoNet support: http://locobuffer.com/ (PL2303 is a lot cheaper, investigate)\n- Level shifting in S88 with transistors?\n- Two way communication on RAILDATA in S88\n- Analog inputs\n- ESP32 (dev board for now, or consider the MAX322/PL2303 and make it all on board now)\n- Break out remaining pins for extra GPIO/UART/SPI/I2C\n-- Level shift to 5V - room on the board?\n"
- moved on the sheet: C?, D?, J?, R?, SW?, TP?, U?, U?A
