File: FlexSensor/FlexSensor.sch (KiCad schematic (older format))
At the start: 222 parts

Commit message: Removed GPIO pins. Used the pins to eliminate SPI in (MOSI). Rearranged SPI pins to the native pins so they can bypass the matrix.
Parts:
- removed C?: 100nF, symbol Device:C_Small
- removed D?: LED_CRGB, symbol Device:LED_CRGB
- removed D?: 1N5819, Diode_THT:D_DO-201AD_P15.24mm_Horizontal, symbol Diode:1N5821
- removed D?: 1N4007, symbol Device:D
- removed J?: GPIO, symbol Connector:Conn_01x06_Male
- removed R?: 36K, symbol Device:R
- removed U?: 74HC165, symbol 74xx:74LS165
- removed U?: 74HCT4053, symbol Trainiot:74HCT4053
- added D?: LED_ARGB, symbol Device:LED_ARGB
- added Q? (x2): Q_PMOS_GDS, symbol Device:Q_PMOS_GDS
- added R? (x2): 100K, symbol Device:R
Connections:
- net GPIO_1 is gone; now on net ~S88_IN_CLK: U?.27 (IO16)
- net GPIO_2 is gone; now on net SPI_CLK: U?.13 (IO14)
- net GPIO_3 is gone; now on net ~S88_OUT_DATA: U?.14 (IO12)
- net GPIO_4 is gone; now on net ~S88_IN_DATA: U?.28 (IO17)
- net +3V3: now also D?.1 (A)
- net GND: now also Q?.1 (G), R?.1
- net SPI_CLK: no longer U?.23 (IO15)
- net USB5V: now also Q?.3 (S)
- net ~S88_IN_DATA: no longer U?.6 (QG)
- net ~S88_IN_LOAD: now also U?.24 (IO2)
- net ~S88_OUT_LOAD: now also U?.6 (QG); no longer U?.7 (QH)
- net ~SPI_SS: now also U?.23 (IO15); no longer U?.24 (IO2)
- net at R?.1: now also D?.2 (RK)
- net at R?.1: now also D?.3 (GK)
- net at R?.1: now also D?.4 (BK)
- net at J?.1 (Pin_1): now also Q?.3 (S), R?.2, R?.2
- net at C?.1, C?.1, C?.1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: now also Q?.2 (D), Q?.2 (D)
- net at U?.11 (S1): now also R?.1
- net at R?.2, U?.13 (1Y1): no longer R?.1
- net MISO_AND_REVISION renamed BUTTON_AND_REVISION
- net BUTTON_AND_REVISION: now also R?.1
- new net: Q?.1 (G), R?.1
- no-connect marks 27 -> 26
Other:
- note removed: "GPIO"
- note removed: "Too big voltage drop for 3.3V regulator?\nWant to favor external 5V over USB 5V - maybe with a mosfet closed when external power is available."
- moved on the sheet: C?, R?, SW?, U?, U?A
