File: FlexSensor/FlexSensor.sch (KiCad schematic (older format))
At the start: 219 parts

Commit message: Added missing ground to 1117 3v3. Updated to KiCad 5.
Parts:
- removed R?: 820K, symbol Device:R
- removed R?: 68K, symbol Device:R
- removed TP?: Test_Point, symbol Connector:Test_Point
- removed U? (x2): LM6132, symbol Amplifier_Operational:LM358
- added U? (x2): LM358, symbol Amplifier_Operational:LM358
Connections:
- net labels added: 24V
Other:
- note removed: "0-1.6V"
Changed lines of the file:
@@
 Text Notes 1450 4750 0    200  ~ 40
 Demultiplexer
-Text GLabel 11350 21000 0    50   Input ~ 0
+Text GLabel 11700 21500 0    50   Input ~ 0
 ANALOG
-$Comp
-L Device:R R?
-U 1 1 5D06ABBF
-P 11650 21250
-F 0 "R?" H 11720 21296 50  0000 L CNN
-F 1 "820K" V 11650 21250 50  0000 C CNN
-F 2 "" V 11580 21250 50  0001 C CNN
-F 3 "~" H 11650 21250 50  0001 C CNN
-	1    11650 21250
-	1    0    0    -1
-$EndComp
-$Comp
-L Device:R R?
-U 1 1 5D06ACF4
-P 11650 21750
-F 0 "R?" H 11720 21796 50  0000 L CNN
-F 1 "68K" V 11650 21750 50  0000 C CNN
-F 2 "" V 11580 21750 50  0001 C CNN
-F 3 "~" H 11650 21750 50  0001 C CNN
-	1    11650 21750
-	1    0    0    -1
-$EndComp
-Wire Wire Line
-	11650 21900 11650 22000
-$Comp
-L power:GND #PWR?
-U 1 1 5D14CB08
-P 11650 22000
-F 0 "#PWR?" H 11650 21750 50  0001 C CNN
-F 1 "GND" H 11800 21950 50  0001 C TNN
-F 2 "" H 11650 22000 50  0001 C CNN
-F 3 "" H 11650 22000 50  0001 C CNN
-	1    11650 22000
-	1    0    0    -1
-$EndComp
-$Comp
-L Amplifier_Operational:LM358 U?
-U 1 1 5D14CF1A
-P 14550 21700
-F 0 "U?" H 14550 21850 50  0000 L CNN
-F 1 "LM6132" H 14500 21500 50  0000 L CNN
-F 2 "" H 14550 21700 50  0001 C CNN
-F 3 "http://www.ti.com/lit/ds/symlink/lm358.pdf" H 14550 21700 50  0001 C CNN
-	1    14550 21700
-	1    0    0    -1
-$EndComp
 Wire Wire Line
 	14850 21700 14950 21700
-$Comp
-L Amplifier_Operational:LM358 U?
-U 1 1 5D40BB93
-P 12950 21600
-F 0 "U?" H 12950 21750 50  0000 L CNN
-F 1 "LM6132" H 12900 21400 50  0000 L CNN
-F 2 "" H 12950 21600 50  0001 C CNN
-F 3 "http://www.ti.com/lit/ds/symlink/lm358.pdf" H 12950 21600 50  0001 C CNN
-	1    12950 21600
-	1    0    0    -1
-$EndComp
-Wire Wire Line
-	11650 21400 11650 21500
-Wire Wire Line
-	11650 21000 11650 21100
 Wire Wire Line
 	12650 21500 12150 21500
-Connection ~ 11650 21500
-Wire Wire Line
-	11650 21500 11650 21600
 $Comp
 L Regulator_SwitchedCapacitor:ICL7660 U?
@@
 Wire Wire Line
 	12850 21000 12850 21300
-Wire Wire Line
-	12450 21000 12450 20900
 Connection ~ 12450 21000
-$Comp
-L power:+3V3 #PWR?
-U 1 1 5C40C0B1
-P 12450 20900
-F 0 "#PWR?" H 12450 20750 50  0001 C CNN
-F 1 "+3V3" H 12465 21073 50  0000 C CNN
-F 2 "" H 12450 20900 50  0001 C CNN
-F 3 "" H 12450 20900 50  0001 C CNN
-	1    12450 20900
-	1    0    0    -1
-$EndComp
 Wire Wire Line
 	13250 21600 13400 21600
@@
 Wire Wire Line
 	12550 21700 12650 21700
-Wire Wire Line
-	11350 21000 11650 21000
 $Comp
 L Device:C_Small C?
@@
 Connection ~ 12150 21500
 Wire Wire Line
-	12150 21500 11650 21500
-Wire Wire Line
 	12150 21850 12150 22000
 $Comp
@@
 $EndComp
 $Comp
-L Connector:Test_Point TP?
-U 1 1 5CC9E626
-P 11650 21000
-F 0 "TP?" H 11600 21200 50  0000 L CNN
-F 1 "Test_Point" H 11708 21029 50  0001 L CNN
-F 2 "" H 11850 21000 50  0001 C CNN
-F 3 "~" H 11850 21000 50  0001 C CNN
-	1    11650 21000
-	1    0    0    -1
-$EndComp
-Connection ~ 11650 21000
-$Comp
 L Device:R R?
 U 1 1 5CD91927
@@
 +0.2V
 Wire Wire Line
-	13600 21400 13600 21050
-Wire Wire Line
 	13600 21400 13700 21400
 $Comp
-L power:+3V3 #PWR?
-U 1 1 5D24A1FC
-P 13600 21050
-F 0 "#PWR?" H 13600 20900 50  0001 C CNN
-F 1 "+3V3" H 13615 21223 50  0000 C CNN
-F 2 "" H 13600 21050 50  0001 C CNN
-F 3 "" H 13600 21050 50  0001 C CNN
-	1    13600 21050
-	1    0    0    -1
-$EndComp
-Text Notes 11800 21050 0    50   ~ 0
-0-1.6V
-$Comp
 L Device:R R?
 U 1 1 5D24B321
@@
 Wire Wire Line
 	8150 1900 8150 2000
+$Comp
+L Amplifier_Operational:LM358 U?
+U 1 1 5B3667E6
+P 12950 21600
+F 0 "U?" H 13291 21646 50  0000 L CNN
+F 1 "LM358" H 13291 21555 50  0000 L CNN
+F 2 "" H 12950 21600 50  0001 C CNN
+F 3 "http://www.ti.com/lit/ds/symlink/lm358.pdf" H 12950 21600 50  0001 C CNN
+	1    12950 21600
+	1    0    0    -1
+$EndComp
+Wire Wire Line
+	12450 20750 12450 21000
+Text GLabel 12400 20750 0    50   Input ~ 0
+24V
+Wire Wire Line
+	12400 20750 12450 20750
+Wire Wire Line
+	12850 21000 13600 21000
+Wire Wire Line
+	13600 21000 13600 21400
+Connection ~ 12850 21000
+$Comp
+L Amplifier_Operational:LM358 U?
+U 1 1 5B6CE2B3
+P 14550 21700
+F 0 "U?" H 14891 21746 50  0000 L CNN
+F 1 "LM358" H 14891 21655 50  0000 L CNN
+F 2 "" H 14550 21700 50  0001 C CNN
+F 3 "http://www.ti.com/lit/ds/symlink/lm358.pdf" H 14550 21700 50  0001 C CNN
+	1    14550 21700
+	1    0    0    -1
+$EndComp
+Wire Wire Line
+	11700 21500 12150 21500
+Text GLabel 10800 1700 2    50   Output ~ 0
+24V
+Wire Wire Line
+	10550 1950 10550 1700
+Wire Wire Line
+	10550 1700 10800 1700
+Connection ~ 10550 1950
+Wire Wire Line
+	5050 3300 5050 3400
 Wire Bus Line
 	3350 14400 4950 14400
@@
 Wire Bus Line
 	4950 5150 4950 14400
+$Comp
+L power:GND #PWR?
+U 1 1 5B9EBAD0
+P 5050 3400
+F 0 "#PWR?" H 5050 3150 50  0001 C CNN
+F 1 "GND" H 5200 3350 50  0001 C TNN
+F 2 "" H 5050 3400 50  0001 C CNN
+F 3 "" H 5050 3400 50  0001 C CNN
+	1    5050 3400
+	1    0    0    -1
+$EndComp
 $EndSCHEMATC

Commit message: Redesigned power/attenuation to no longer require a negative rail at the cost of possible minor current feedback to sensor.
Parts:
- removed C? (x4): 330nF, symbol Device:C_Small
- removed C? (x3): 10μF, symbol Device:CP
- removed C?: 100µF, symbol Device:CP
- removed C?: 4.7µF, symbol Device:CP
- removed C? (x2): 22μF, symbol Device:C_Small
- removed C?: NC (2.2uF), symbol Device:CP
- removed C? (x5): 100nF, symbol Device:C_Small
- removed C? (x5): NC, symbol Device:C_Small
- removed D?: 1N5821, Diode_THT:D_DO-201AD_P15.24mm_Horizontal, symbol Diode:1N5821
- removed J?: 5-15VDC, symbol Connector:Screw_Terminal_01x02
- removed L?: 22μH, symbol Device:L
- removed Q? (x2): Q_PMOS_GDS, symbol Device:Q_PMOS_GDS
- removed R?: 9.1, symbol Device:R
- removed R?: 270, symbol Device:R
- removed R?: 470K, symbol Device:R
- removed R?: 12K, symbol Device:R
- removed R? (x6): 10K, symbol Device:R
- removed R? (x2): 100K, symbol Device:R
- removed R? (x2): 180K, symbol Device:R
- removed TP? (x6): Test_Point, symbol Connector:Test_Point
- removed U?: ICL7660, symbol Regulator_SwitchedCapacitor:ICL7660
- removed U?: MT3608, symbol Trainiot:MT3608
- removed U? (x2): LM358, symbol Amplifier_Operational:LM358
- removed U?: LM78L05, symbol Trainiot:LM78L05
- removed U?: LD1117S33TR_SOT223, Package_TO_SOT_SMD:SOT-223-3_TabPin2, symbol Regulator_Linear:LD1117S33TR_SOT223
- removed U?: LM7820, Package_TO_SOT_THT:TO-220-3_Vertical, symbol Regulator_Linear:LM7805_TO220
- removed U? (x2): LM6132, symbol Amplifier_Operational:LM358
- removed U?: MCP42010, symbol Potentiometer_Digital:MCP42010
- added C115, C118, C123: NC, symbol Device:C_Small
- added C116, C119, C135: 100nF, symbol Device:C_Small
- added C120, C122, C151: 100µF, symbol Device:CP
- added C125, C131: 22μF, symbol Device:C_Small
- added C126: 680µF, symbol Device:CP
- added C139: 220µF, symbol Device:CP
- added C141: 220µF/NP, symbol Device:CP
- added C143: 330nF, symbol Device:C_Small
- added C146: 10µF, symbol Device:CP
- added D102, D103, D104, D105, D106, D107, D109, D110: 1N5821, Diode_THT:D_DO-201AD_P15.24mm_Horizontal, symbol Diode:1N5821
- added FB101: ~, symbol Device:Ferrite_Bead_Small
- added J113: 7-20VDC, symbol Connector:Screw_Terminal_01x02
- added L101: 22μH, symbol Device:L
- added L102: 33μH, symbol Device:L
- added L103: 3μH/NP, symbol Device:L
- added R132: 820K, symbol Device:R
- added R133: 68K, symbol Device:R
- added R140, R164: 2.2K, symbol Device:R
- added R141, R143: 10K, symbol Device:R
- added R142, R145, R151: 1K, symbol Device:R
- added R148: 470K, symbol Device:R
- added R149: 12K, symbol Device:R
- added R150, R152, R158, R159: NP, symbol Device:R
- added R153: 3.3K, symbol Device:R
- added R160: 0, symbol Device:R
- added R165: 33K, symbol Device:R
- added TP101, TP102, TP103, TP104, TP105, TP106: Test_Point, symbol Connector:Test_Point
- added TP107, TP108, TP109, TP110, TP111, TP113: TestPoint, symbol Connector:TestPoint
- added U117: MCP42010, symbol Potentiometer_Digital:MCP42010
- added U119: MCP6001R, Package_TO_SOT_SMD:SOT-23-5, symbol Amplifier_Operational:MCP6001R
- added U122: MT3608, symbol Trainiot:MT3608
- added U123: LM2596S-ADJ, Package_TO_SOT_SMD:TO-263-5_TabPin3, symbol Regulator_Switching:LM2596S-ADJ
- added U126: LM317_3PinPackage, symbol Regulator_Linear:LM317_3PinPackage
- added unit 3 of U127
- added U130: LM1117-3.3, symbol Regulator_Linear:LM1117-3.3
- gave numbers to parts that had none: 152
Connections:
- net labels removed: -3V3, 24V
- wire segments 1093 -> 1075
- no-connect marks 26 -> 24
Other:
- note added: "0.32 - 1.81V offset"
- note added: "Gain: -0.9 to -10"
- note added: "Optional filter"
- note added: "Target voltage: 0 - 1.6"
- note added: "Target voltage: 0.2 - 1.8"
- note removed: "+0.2V"
- note removed: "-offset"
- note removed: "Check diode choice\nin MT3608 datasheet"
- moved on the sheet: C101, C102, C103, C104, C105, C106, C107, C108, C109, C110, C111, C112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

Commit message: Initial foot print assigments
Parts:
- removed U108, U109, U115: LM339, symbol Comparator:LM339
- removed U132: LM393, symbol Comparator:LM393
- added unit 2 of U107
- added unit 3 of U107
- added unit 4 of U107
- added unit 5 of U107
- added unit 2 of U127
- C101, C102, C103, C104, C105, C106, C107, C108, C109, C110, C111, C112, C113, C114, C115, C116, C117, C118, C119, C120, C121, C122, C123, C124, C127, C128, C129, C130, C132, C133, C134, C135, C136, C137, C138, C140, C142, C143, C144, C145, C148: footprint (none) -> Capacitors_SMD:C_0603
- C125, C131, C146: footprint (none) -> Capacitors_THT:CP_Radial_D5.0mm_P2.00mm
- C126: footprint (none) -> Capacitors_THT:CP_Radial_D10.0mm_P5.00mm
- C139: footprint (none) -> Capacitors_THT:CP_Radial_D8.0mm_P3.80mm
- C141: value 220µF/NP -> 180µF/NP; footprint (none) -> Capacitors_THT:CP_Radial_D8.0mm_P3.80mm
- C151: footprint (none) -> Capacitors_THT:CP_Radial_D7.5mm_P2.50mm
- D101: footprint (none) -> LEDs:LED_D5.0mm-4
- D108, D111, D112, D113: footprint (none) -> LEDs:LED_0603
- FB101, L104, R101, R102, R103, R104, R105, R106, R107, R108, R109, R110, R111, R112, R113, R114, R115, R116, R117, R118, R119, R120, R121, R122, R123, R124, R125, R126, R127, R128, R129, R130, R131, R132, R133, R134, R135, R136, R137, R138, R139, R140, R141, R142, R143, R144, R145, R146, R147, R148, R149, R150, R151, R152, R153, R154, R155, R156, R157, R158, R159, R160, R161, R162, R163, R164, R165, R166, R167, R168, R169, R170, R171, R172, R173, R174, R175, R176, R177, R178, R179, R180: footprint (none) -> Resistors_SMD:R_0603
- J101, J112: footprint (none) -> Connectors:RJ45_8
- J102, J111, J119: footprint (none) -> Pin_Headers:Pin_Header_Straight_1x06_Pitch2.54mm
- J103, J104, J105, J107, J108, J109: footprint (none) -> Connectors_Phoenix:PhoenixContact_MCV-G_08x3.50mm_Vertical
- J106, J110: footprint (none) -> Connectors_Phoenix:PhoenixContact_MCV-G_06x3.50mm_Vertical
- J113: footprint (none) -> Connectors_Terminal_Blocks:TerminalBlock_bornier-2_P5.08mm
- J114: footprint (none) -> Connectors:USB_Micro-B
- J115, J116, J117, J118: footprint (none) -> Connectors:RJ12_E
- J120: footprint (none) -> Connectors:RJ45_TRANSFO
- L101, L102, L103: footprint (none) -> Inductors:Inductor_Taiyo-Yuden_NR-40xx
- SW101, SW102: footprint (none) -> Buttons_Switches_THT:SW_PUSH_6mm
- SW103: footprint (none) -> Buttons_Switches_SMD:SW_DIP_x1_W5.08mm_Slide_Copal_CHS-A
- TP101, TP102, TP103, TP104, TP105, TP106, TP107, TP108, TP109, TP110, TP111, TP113: footprint (none) -> Measurement_Points:Test_Point
- U101: footprint (none) -> Housings_SOIC:SOIC-18W_7.5x11.6mm_Pitch1.27mm
- U102, U103, U104, U105, U106, U110, U111, U112, U113, U114, U118: footprint (none) -> Housings_SOIC:SOIC-16_3.9x9.9mm_Pitch1.27mm
- U107, U116: footprint (none) -> Housings_SOIC:SOIC-14_3.9x8.7mm_Pitch1.27mm
- U117: footprint (none) -> Housings_SSOP:TSSOP-14_4.4x5mm_Pitch0.65mm
- U120: footprint (none) -> Housings_SSOP:SOP-16_4.4x10.4mm_Pitch1.27mm
- U121: footprint (none) -> Crystals:Crystal_SMD_3225-4pin_3.2x2.5mm_HandSoldering
- U122: footprint (none) -> TO_SOT_Packages_SMD:SOT-23-6
- U125: footprint (none) -> Housings_DFN_QFN:QFN-28-1EP_5x5mm_Pitch0.5mm
- U126, U130: footprint (none) -> TO_SOT_Packages_SMD:SOT-223
- U127: footprint (none) -> Housings_SOIC:HTSOP-8-1EP_3.9x4.9mm_Pitch1.27mm
- U128: footprint (none) -> Housings_SOIC:SOIC-8_3.9x4.9mm_Pitch1.27mm
- U129: footprint (none) -> Trainiot:ESP32-WROOM

Commit message: Updated diodes to SMD
Parts:
- removed D102, D103, D104, D105, D106, D107, D109, D110: 1N5821, Diode_THT:D_DO-201AD_P15.24mm_Horizontal, symbol Diode:1N5821
- added D102, D107, D109, D110: SS12, Diodes_SMD:D_SMA, symbol Device:D_Schottky
- added D103, D104, D105: SS13, Diodes_SMD:D_SMA, symbol Device:D_Schottky
- added D106: SS34, Diodes_SMD:D_SMA, symbol Device:D_Schottky
- D101: footprint LEDs:LED_D5.0mm-4 -> LEDs:LED_Cree-PLCC4_2x2mm_CW
Changed lines of the file:
@@
 F 0 "D101" H 9600 4033 50  0000 C CNN
 F 1 "LED_ARGB" H 9600 4124 50  0000 C CNN
-F 2 "LEDs:LED_D5.0mm-4" H 9600 4450 50  0001 C CNN
+F 2 "LEDs:LED_Cree-PLCC4_2x2mm_CW" H 9600 4450 50  0001 C CNN
 F 3 "~" H 9600 4450 50  0001 C CNN
 	1    9600 4500
@@
 Text Notes 10900 20300 0    200  ~ 40
 Power
-$Comp
-L Diode:1N5821 D109
-U 1 1 5C1FAD11
-P 16850 22100
-F 0 "D109" H 16900 22000 50  0000 R CNN
-F 1 "1N5821" H 17000 22250 50  0000 R CNN
-F 2 "Diode_THT:D_DO-201AD_P15.24mm_Horizontal" H 16850 21925 50  0001 C CNN
-F 3 "http://www.vishay.com/docs/88526/1n5820.pdf" H 16850 22100 50  0001 C CNN
-	1    16850 22100
-	-1   0    0    1
-$EndComp
 Text GLabel 11150 22100 0    50   Input ~ 0
 USB5V
@@
 Wire Wire Line
 	13500 23250 13700 23250
-$Comp
-L Diode:1N5821 D107
-U 1 1 5CD3863B
-P 14900 23500
-F 0 "D107" V 14950 23400 50  0000 R CNN
-F 1 "1N5821" V 15050 23350 50  0000 R CNN
-F 2 "Diode_THT:D_DO-201AD_P15.24mm_Horizontal" H 14900 23325 50  0001 C CNN
-F 3 "http://www.vishay.com/docs/88526/1n5820.pdf" H 14900 23500 50  0001 C CNN
-	1    14900 23500
-	0    1    1    0
-$EndComp
 Wire Wire Line
 	14900 23350 14900 23250
@@
 	16300 23050 16300 23250
 Connection ~ 16300 23250
-$Comp
-L Diode:1N5821 D110
-U 1 1 5F19F9B2
-P 16850 23250
-F 0 "D110" H 16900 23150 50  0000 R CNN
-F 1 "1N5821" H 17000 23350 50  0000 R CNN
-F 2 "Diode_THT:D_DO-201AD_P15.24mm_Horizontal" H 16850 23075 50  0001 C CNN
-F 3 "http://www.vishay.com/docs/88526/1n5820.pdf" H 16850 23250 50  0001 C CNN
-	1    16850 23250
-	-1   0    0    1
-$EndComp
 Wire Wire Line
 	16700 23250 16300 23250
-$Comp
-L Diode:1N5821 D105
-U 1 1 5F7A3E3F
-P 12000 23050
-F 0 "D105" H 12050 22950 50  0000 R CNN
-F 1 "1N5821" H 12150 23200 50  0000 R CNN
-F 2 "Diode_THT:D_DO-201AD_P15.24mm_Horizontal" H 12000 22875 50  0001 C CNN
-F 3 "http://www.vishay.com/docs/88526/1n5820.pdf" H 12000 23050 50  0001 C CNN
-	1    12000 23050
-	-1   0    0    1
-$EndComp
 Wire Wire Line
 	11400 23050 11750 23050
@@
 Wire Wire Line
 	13750 20700 13650 20700
-$Comp
-L Diode:1N5821 D106
-U 1 1 60CB6750
-P 14000 20700
-F 0 "D106" H 14050 20600 50  0000 R CNN
-F 1 "1N5821" H 14150 20850 50  0000 R CNN
-F 2 "Diode_THT:D_DO-201AD_P15.24mm_Horizontal" H 14000 20525 50  0001 C CNN
-F 3 "http://www.vishay.com/docs/88526/1n5820.pdf" H 14000 20700 50  0001 C CNN
-	1    14000 20700
-	-1   0    0    1
-$EndComp
 Wire Wire Line
 	13850 20700 13750 20700
@@
 	12500 20700 12850 20700
 Connection ~ 12850 20700
-$Comp
-L Diode:1N5821 D103
-U 1 1 635B7A77
-P 11550 20700
-F 0 "D103" H 11600 20600 50  0000 R CNN
-F 1 "1N5821" H 11700 20850 50  0000 R CNN
-F 2 "Diode_THT:D_DO-201AD_P15.24mm_Horizontal" H 11550 20525 50  0001 C CNN
-F 3 "http://www.vishay.com/docs/88526/1n5820.pdf" H 11550 20700 50  0001 C CNN
-	1    11550 20700
-	-1   0    0    1
-$EndComp
 Wire Wire Line
 	11300 20700 11300 22100
@@
 	11700 20700 11750 20700
 Connection ~ 12500 20700
-$Comp
-L Diode:1N5821 D104
-U 1 1 6467B980
-P 11750 21050
-F 0 "D104" V 11750 21200 50  0000 R CNN
-F 1 "1N5821" V 11850 21400 50  0000 R CNN
-F 2 "Diode_THT:D_DO-201AD_P15.24mm_Horizontal" H 11750 20875 50  0001 C CNN
-F 3 "http://www.vishay.com/docs/88526/1n5820.pdf" H 11750 21050 50  0001 C CNN
-	1    11750 21050
-	0    1    1    0
-$EndComp
 Wire Wire Line
 	11750 21200 11750 23050
@@
 Text Notes 10550 13250 0    50   ~ 0
 0.32 - 1.81V offset
-$Comp
-L Diode:1N5821 D102
-U 1 1 5C3FC151
-P 10300 10800
-F 0 "D102" H 10350 10700 50  0000 R CNN
-F 1 "1N5821" H 10450 10950 50  0000 R CNN
-F 2 "Diode_THT:D_DO-201AD_P15.24mm_Horizontal" H 10300 10625 50  0001 C CNN
-F 3 "http://www.vishay.com/docs/88526/1n5820.pdf" H 10300 10800 50  0001 C CNN
-	1    10300 10800
-	0    1    1    0
-$EndComp
 Connection ~ 10300 11300
 Wire Wire Line
@@
 Wire Bus Line
 	4950 1600 4950 10850
+$Comp
+L Device:D_Schottky D103
+U 1 1 5C15108A
+P 11550 20700
+F 0 "D103" H 11550 20484 50  0000 C CNN
+F 1 "SS13" H 11550 20575 50  0000 C CNN
+F 2 "Diodes_SMD:D_SMA" H 11550 20700 50  0001 C CNN
+F 3 "~" H 11550 20700 50  0001 C CNN
+	1    11550 20700
+	-1   0    0    1
+$EndComp
+$Comp
+L Device:D_Schottky D104
+U 1 1 5C152654
+P 11750 21050
+F 0 "D104" V 11704 21129 50  0000 L CNN
+F 1 "SS13" V 11795 21129 50  0000 L CNN
+F 2 "Diodes_SMD:D_SMA" H 11750 21050 50  0001 C CNN
+F 3 "~" H 11750 21050 50  0001 C CNN
+	1    11750 21050
+	0    1    1    0
+$EndComp
+$Comp
+L Device:D_Schottky D105
+U 1 1 5C153AF2
+P 12000 23050
+F 0 "D105" H 12000 22834 50  0000 C CNN
+F 1 "SS13" H 12000 22925 50  0000 C CNN
+F 2 "Diodes_SMD:D_SMA" H 12000 23050 50  0001 C CNN
+F 3 "~" H 12000 23050 50  0001 C CNN
+	1    12000 23050
+	-1   0    0    1
+$EndComp
+$Comp
+L Device:D_Schottky D106
+U 1 1 5C15478C
+P 14000 20700
+F 0 "D106" H 14000 20484 50  0000 C CNN
+F 1 "SS34" H 14000 20575 50  0000 C CNN
+F 2 "Diodes_SMD:D_SMA" H 14000 20700 50  0001 C CNN
+F 3 "~" H 14000 20700 50  0001 C CNN
+	1    14000 20700
+	-1   0    0    1
+$EndComp
+$Comp
+L Device:D_Schottky D110
+U 1 1 5C154A6D
+P 16850 23250
+F 0 "D110" H 16850 23034 50  0000 C CNN
+F 1 "SS12" H 16850 23125 50  0000 C CNN
+F 2 "Diodes_SMD:D_SMA" H 16850 23250 50  0001 C CNN
+F 3 "~" H 16850 23250 50  0001 C CNN
+	1    16850 23250
+	-1   0    0    1
+$EndComp
+$Comp
+L Device:D_Schottky D109
+U 1 1 5C154E55
+P 16850 22100
+F 0 "D109" H 16850 21884 50  0000 C CNN
+F 1 "SS12" H 16850 21975 50  0000 C CNN
+F 2 "Diodes_SMD:D_SMA" H 16850 22100 50  0001 C CNN
+F 3 "~" H 16850 22100 50  0001 C CNN
+	1    16850 22100
+	-1   0    0    1
+$EndComp
+$Comp
+L Device:D_Schottky D107
+U 1 1 5C15A58B
+P 14900 23500
+F 0 "D107" V 14854 23579 50  0000 L CNN
+F 1 "SS12" V 14945 23579 50  0000 L CNN
+F 2 "Diodes_SMD:D_SMA" H 14900 23500 50  0001 C CNN
+F 3 "~" H 14900 23500 50  0001 C CNN
+	1    14900 23500
+	0    1    1    0
+$EndComp
+$Comp
+L Device:D_Schottky D102
+U 1 1 5C15B4DA
+P 10300 10800
+F 0 "D102" V 10254 10879 50  0000 L CNN
+F 1 "SS12" V 10345 10879 50  0000 L CNN
+F 2 "Diodes_SMD:D_SMA" H 10300 10800 50  0001 C CNN
+F 3 "~" H 10300 10800 50  0001 C CNN
+	1    10300 10800
+	0    1    1    0
+$EndComp
 $EndSCHEMATC
